File: fos12_ma/aufgaben/ladung_c/ladung_c.kicad_sch (KiCad schematic)
At the start: 3 parts

Commit message: Lösungsvorschläge hinzugefügt
Parts:
- C1: value 560u -> 470u
- R1: value 1k2 -> 2k2
- V1: value 14,5 -> 12
Changed lines of the file:
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@@
 			)
 		)
-		(property "Value" "14,5"
+		(property "Value" "12"
 			(at 41.91 86.2301 0)
 			(effects
@@
 			)
 		)
-		(property "Value" "1k2"
+		(property "Value" "2k2"
 			(at 48.26 72.39 90)
 			(effects
@@
 			)
 		)
-		(property "Value" "560u"
+		(property "Value" "470u"
 			(at 60.96 87.6299 0)
 			(effects
