File: fos12_ma/aufgaben/schaltung4/schaltung5/schaltung5.kicad_sch (KiCad schematic)
At the start: 8 parts

Commit message: Korrekturen und Ergänzung
Parts:
- removed I1: 120mA, symbol Simulation_SPICE:IDC
- added V3: 5, symbol Simulation_SPICE:VDC
- R_CE1: value 70 -> 250
Connections:
- net GND: now also V3.2; no longer R_CE1.2
- new net: R_CE1.2, V3.1
Other:
- note added: "U_CE=5 V, I_C=20 mA, I_B = 50 uA"
Changed lines of the file:
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@@
+	)
+	(junction
+		(at 114.3 88.9)
+		(diameter 0)
+		(color 0 0 0 0)
 	)
 	(junction
@@
 	)
 	(junction
-		(at 114.3 88.9)
-		(diameter 0)
-		(color 0 0 0 0)
-	)
-	(junction
 		(at 101.6 88.9)
 		(diameter 0)
@@
 	(wire
 		(pts
+			(xy 82.55 77.47) (xy 82.55 88.9)
+		)
+		(stroke
+			(width 0)
+			(type default)
+		)
+	)
+	(wire
+		(pts
 			(xy 101.6 88.9) (xy 114.3 88.9)
 		)
@@
 	(wire
 		(pts
-			(xy 82.55 77.47) (xy 82.55 88.9)
-		)
-		(stroke
-			(width 0)
-			(type default)
-		)
-	)
-	(wire
-		(pts
-			(xy 146.05 88.9) (xy 114.3 88.9)
+			(xy 114.3 77.47) (xy 114.3 78.74)
 		)
 		(stroke
@@
 	(wire
 		(pts
-			(xy 101.6 69.85) (xy 101.6 63.5)
-		)
-		(stroke
-			(width 0)
-			(type default)
-		)
-	)
-	(wire
-		(pts
 			(xy 69.85 44.45) (xy 114.3 44.45)
 		)
@@
 	(wire
 		(pts
+			(xy 114.3 88.9) (xy 146.05 88.9)
+		)
+		(stroke
+			(width 0)
+			(type default)
+		)
+	)
+	(wire
+		(pts
 			(xy 38.1 60.96) (xy 69.85 60.96)
 		)
@@
 	(wire
 		(pts
-			(xy 114.3 77.47) (xy 114.3 88.9)
-		)
-		(stroke
-			(width 0)
-			(type default)
-		)
-	)
-	(wire
-		(pts
 			(xy 38.1 80.01) (xy 38.1 88.9)
 		)
@@
 			(width 0)
 			(type default)
+		)
+	)
+	(text "U_CE=5 V,\nI_C=20 mA,\nI_B = 50 uA"
+		(exclude_from_sim no)
+		(at 131.826 73.406 0)
+		(effects
+			(font
+				(size 1.27 1.27)
+			)
 		)
 	)
@@
 			)
 		)
-		(property "Value" "70"
+		(property "Value" "250"
 			(at 116.84 74.9299 0)
 			(effects
@@
 	)
 	(symbol
-		(lib_id "Simulation_SPICE:IDC")
-		(at 101.6 74.93 0)
+		(lib_id "Simulation_SPICE:VDC")
+		(at 114.3 83.82 0)
 		(unit 1)
 		(exclude_from_sim no)
@@
 		(dnp no)
 		(fields_autoplaced yes)
-		(property "Reference" "I1"
-			(at 105.41 73.6599 0)
-			(effects
-				(font
-					(size 1.27 1.27)
-				)
-				(justify left)
-			)
-		)
-		(property "Value" "120mA"
-			(at 105.41 76.1999 0)
+		(property "Reference" "V3"
+			(at 118.11 82.4048 0)
+			(effects
+				(font
+					(size 1.27 1.27)
+				)
+				(justify left)
+			)
+		)
+		(property "Value" "5"
+			(at 118.11 84.9448 0)
 			(effects
 				(font
@@
 		)
 		(property "Footprint" ""
-			(at 101.6 74.93 0)
+			(at 114.3 83.82 0)
 			(effects
 				(font
@@
 		)
 		(property "Datasheet" "https://ngspice.sourceforge.io/docs/ngspice-html-manual/manual.xhtml#sec_Independent_Sources_for"
-			(at 101.6 74.93 0)
-			(effects
-				(font
-					(size 1.27 1.27)
-				)
-				(hide yes)
-			)
-		)
-		(property "Description" "Current source, DC"
-			(at 101.6 74.93 0)
+			(at 114.3 83.82 0)
+			(effects
+				(font
+					(size 1.27 1.27)
+				)
+				(hide yes)
+			)
+		)
+		(property "Description" "Voltage source, DC"
+			(at 114.3 83.82 0)
 			(effects
 				(font
@@
 		)
 		(property "Sim.Pins" "1=+ 2=-"
-			(at 101.6 74.93 0)
+			(at 114.3 83.82 0)
 			(effects
 				(font
@@
 		)
 		(property "Sim.Type" "DC"
-			(at 101.6 74.93 0)
-			(effects
-				(font
-					(size 1.27 1.27)
-				)
-				(hide yes)
-			)
-		)
-		(property "Sim.Device" "I"
-			(at 101.6 74.93 0)
-			(effects
-				(font
-					(size 1.27 1.27)
-				)
-				(hide yes)
-			)
+			(at 114.3 83.82 0)
+			(effects
+				(font
+					(size 1.27 1.27)
+				)
+				(hide yes)
+			)
+		)
+		(property "Sim.Device" "V"
+			(at 114.3 83.82 0)
+			(effects
+				(font
+					(size 1.27 1.27)
+				)
+				(justify left)
+				(hide yes)
+			)
+		)
+		(pin "1"
 		)
 		(pin "2"
-		)
-		(pin "1"
 		)
 		(instances
 			(project ""
 				(path "/e6463b6c-a4fb-4868-881c-bf66560d0c1d"
-					(reference "I1")
+					(reference "V3")
 					(unit 1)
 				)
